File: Voltage Source/Voltage Source/Voltage Source.kicad_sch (KiCad schematic)
At the start: 40 parts, among them J1 WQP518MA, J2 WQP518MA, J3 Conn_01x01_Male, J4 Conn_01x01_Male, J5 Conn_02x05_Odd_Even, J6 Conn_02x05_Odd_Even, SW1 SW_DPDT_x2, SW2 SW_DPDT_x2, U1 TL072, U2 LM385BXZ-2.5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

Commit message: Updated Voltage Source to REV 5
Parts:
- added C8: 100n, Capacitor_THT:C_Disc_D4.7mm_W2.5mm_P5.00mm, symbol Device:C
- C1, C4, C6, C7: footprint NSI Footprints:C_Disc_D4mm_W2.6mm_P5.08mm -> Capacitor_THT:C_Disc_D4.7mm_W2.5mm_P5.00mm
- C2, C3: value 10u -> 2.2u
- C5: value 10n -> 100n; footprint NSI Footprints:C_Disc_D4mm_W2.6mm_P5.08mm -> Capacitor_THT:C_Disc_D4.7mm_W2.5mm_P5.00mm
- J1, J2: footprint NSI Footprints:Jack_3.5mm_QingPu_WQP-PJ398SM_Vertical_2HP -> Footprints:QingPu_WQP518MA
- R1, R2: value 3k -> 22k
- R10, R15: value 51k -> 12k
- R13, R8: value 82k -> 20k
- R5, R6: value 100k -> 24k
- RV1, RV2, RV3, RV4, RV5, RV6: footprint NSI Footprints:Potentiometer_TT_67Y_Vertical -> Potentiometer_THT:Potentiometer_Bourns_3296Y_Vertical
- SW1, SW2: footprint NSI Footprints:SW_Taiway_Sub_DPDT -> 2 Specific Footprints:SW_Sub_DPDT
- U1: value TL072 -> LF412
Connections:
- net GND: now also C5.2, C8.1
- net VEE: now also C8.2; no longer C5.2
Other:
- moved on the sheet: C5, U1C

Commit message: changed current limiting resistors and 0V resistors, and cleaned up silk layer
Parts:
- R1: value 22k -> 12k
- R12, R7: value 4.7M -> 10M
- R2: value 22k -> 24k
Changed lines of the file:
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@@
 			)
 		)
-		(property "Value" "22k"
+		(property "Value" "24k"
 			(at 23.368 27.813 0)
 			(show_name no)
@@
 			)
 		)
-		(property "Value" "22k"
+		(property "Value" "12k"
 			(at 19.812 94.107 0)
 			(show_name no)
@@
 			)
 		)
-		(property "Value" "4.7M"
+		(property "Value" "10M"
 			(at 80.01 77.8764 90)
 			(show_name no)
@@
 			)
 		)
-		(property "Value" "4.7M"
+		(property "Value" "10M"
 			(at 80.01 41.0464 90)
 			(show_name no)
